File: wiring/wiring.kicad_sch (KiCad schematic)
At the start: 18 parts

Commit message: updated some connectors and power connections
Parts:
- removed J? (x3): M1 Encoder, symbol Connector:Conn_01x02_Female
- removed J?: M1 ENC PWR, symbol Connector:Conn_01x02_Female
- added J? (x6): Screw_Terminal_01x02, symbol Connector:Screw_Terminal_01x02
- U?: value TB6612FNG -> 426-DRI0044; footprint Package_SO:SSOP-24_5.3x8.2mm_P0.65mm -> (none)
- U?: footprint Sensor_Motion:InvenSense_QFN-24_3x3mm_P0.4mm -> (none)
Connections:
- net 3V3-3 is gone; now on net +5V: U?.6 (+VIO)
- net GND-2 is gone; now on net GND: U?.20 (GND)
- net +5V: now also J?.1 (Pin_1), J?.2 (Pin_2); no longer J?.4 (Pin_4), J?.4 (Pin_4), M?.2 (ENC_PWR), U?.2 (3V3), U?.2 (3V3)
- net ENCA_M1: now also J?.1 (Pin_1); no longer A?.5 (D2), M?.4 (ENC_B)
- net ENCA_M2: now also J?.2 (Pin_2)
- net ENCB_M2: now also J?.1 (Pin_1)
- net GND: now also U?.18 (GND), J?.1 (Pin_1), J?.2 (Pin_2)
- net NEG_M1: now also J?.1 (Pin_1)
- net NEG_M2: now also J?.2 (Pin_2)
- net PWR_M1: now also J?.2 (Pin_2)
- net PWR_M2: now also J?.1 (Pin_1)
- net INT: now reaches A?.7 (D4)
- net PWM renamed RESET
- new net +3V3: J?.4 (Pin_4), J?.4 (Pin_4), U?.2 (3V3), U?.2 (3V3)
- new net ENCB_M1: A?.5 (D2), J?.2 (Pin_2), M?.4 (ENC_B)
- no-connect marks 20 -> 19
Other:
- note added: "Encoder GND"
- note added: "Encoder VCC"
- note added: "IMU"
- note added: "M1 Encoder"
- note added: "M1 PWR"
- note added: "M2 Encoder"
- note added: "M2 PWR"
- note added: "MOTOR CONTROLLER"
- note added: "TOF"
- note added: "switching controllers: https://www.digikey.ca/en/products/filter/power-management-pmic/voltage-regulators-dc-dc-switching-regulators/739?s=N4IgjCBcoCwdIDGUBmBDANgZwKYBoQB7KAbRAGYYB2GciAXQIAcAXKEAZRYCcBLAOwDmIAL4EwYAAxRQySOmz4ipEDEkAOcuoBMIRiFbsufIaPFUqAThlJUmXAWKQy2mJYCsANiogC2z%2B7Sfm5gVAzMbJCcPALCYiAAtLoIcjwArkpOZO56InlAA"
- note removed: "2-ENC 2x5V"
- note removed: "SCREW TERMINAL X 8"
- moved on the sheet: A?, D?, J?, U?
